File: kicad/kicad.kicad_sch (KiCad schematic)
At the start: 44 parts, among them J1 USB_C_Receptacle_USB2.0_16P, J2 Barrel_Jack_MountingPin, Q1 NMOS, Q2 NMOS, SW3 SW_SPST, U1 LD1117S50TR_SOT223, U2 TP5100, U3 HY2120, U4 LD1117S33TR_SOT223, U6 MP2307

Commit message: Completed the PCB
Other:
- note added: "BMS"
- note added: "BUCK CONVERTER"
- note added: "CHARGING CIRCUIT"
- note added: "LDO: 3V3"
- note added: "LDO: 5V"
- note added: "MCU, MODULES & PERIPHERALS"
- note added: "TYPE-C (FOR CODE ONLY)"
- moved on the sheet: BT1, BT2, C1, C10, C19, C2, C23, C24, C25, C26, C3, C4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
