File: kicad/kicad.kicad_sch (KiCad schematic)
At the start: 44 parts, among them J1 USB_C_Receptacle_USB2.0_16P, J2 Barrel_Jack_MountingPin, Q1 NMOS, Q2 NMOS, SW3 SW_SPST, U1 LD1117S50TR_SOT223, U2 TP5100, U3 HY2120, U4 LD1117S33TR_SOT223, U6 MP2307

Commit message: update
Parts:
- removed C25: 12uF, Capacitor_SMD:C_0805_2012Metric_Pad1.18x1.45mm_HandSolder, symbol Device:C
- removed L1: 22uH, Inductor_SMD:L_10.4x10.4_H4.8, symbol Device:L
- added C22: 22 uF, Capacitor_SMD:CP_Elec_5x5.3, symbol Device:C_Polarized
- added U10: CDRH104R-220NC, easyeda2kicad:IND-SMD_L10.2-W10.0_SRR1050HA, symbol easyeda2kicad:CDRH104R-220NC
- BT1: renamed from BT2; Link (none) -> https://hubtronics.in/1s-18650-holder-smd?srsltid=AfmBOor3T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; Price (none) -> 57.82
- BT2: renamed from BT1; Link (none) -> https://hubtronics.in/1s-18650-holder-smd?srsltid=AfmBOor3T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; Price (none) -> 57.82
- C1: renamed from C23; Link (none) -> https://robu.in/product/efvl063ada100m0654-follon-10uf-63v-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; Price (none) -> 2.09
- C2: renamed from C24; value 0.1uF -> 100nF
- C3: renamed from C26; Link (none) -> https://robu.in/product/tcc0805x7r392k500dt-cctc-smt-cerami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; Price (none) -> 0.29
- C4: renamed from C19; Link (none) -> https://robu.in/product/1-month-warranty-262/; Price (none) -> 1.39
- C6: renamed from C5; Link (none) -> http://robu.in/product/tcc0805x7r104k500dt-cctc-smt-ceramic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; Price (none) -> 0.97
- C7: renamed from C6; Link (none) -> https://robu.in/product/10uf-10000nf-25-v-capacitor-0805-sm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; Price (none) -> 3.24
- C8: renamed from C9; Link (none) -> https://robu.in/product/21br61a226me51k-murata-cap-smd-mlcc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; Price (none) -> 9
- D1: renamed from D4; Link (none) -> https://evelta.com/schottky-diode-1a-sma-ss110/; Price (none) -> 2.70
- D2: Link (none) -> https://robu.in/product/0805-surface-mount-led-green-50-pcs/; Price (none) -> 2.62
- D3: Link (none) -> https://robu.in/product/0805-surface-mount-led-red-50-pcs/; Price (none) -> 1.44
- J1: Link (none) -> http://robu.in/product/type-c-31-m-12-hroparts-5a-1-16p-fem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; Price (none) -> 38
- J2: Link (none) -> https://robu.in/product/dc-jack-005/; Price (none) -> 2.23
- L1: renamed from L3; footprint Inductor_SMD:L_10.4x10.4_H4.8 -> easyeda2kicad:IND-SMD_L10.2-W10.0_SRR1050HA; Link (none) -> https://robu.in/product/cdrh104r-10%CE%BCh-power-inductor-p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; Price (none) -> 15
- Q1: Link (none) -> https://robu.in/product/cmn2310m-cmos-smd-mos-sot-23-n-fiel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; Price (none) -> 1.78
- R1: renamed from R23; Link (none) -> https://robu.in/product/yageo-100k-ohm-1-2w-0805-surface-mo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; Price (none) -> 0.54
- R2: renamed from R1; Link (none) -> https://robu.in/product/af0805fr-075k1l-yageo-5-1k%CF%89-%C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; Price (none) -> 1.57
- R3: renamed from R2; Link (none) -> https://robu.in/product/af0805fr-075k1l-yageo-5-1k%CF%89-%C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; Price (none) -> 1.57
- R4: renamed from R28; Link (none) -> https://robu.in/product/ac0805jr-076k8l-yageo-res-thick-fil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; Price (none) -> 0.87
- R5: renamed from R26; Link (none) -> https://robu.in/product/rc0805fr-0710kl-yageo-res-thick-fil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; Price (none) -> 0.80
- R6: renamed from R24; Link (none) -> https://robu.in/product/ac0805fr-0730k9l-yageo-125mw-thick-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; Price (none) -> 1.13
- R7: Link (none) -> https://robu.in/product/1k-ohm-1-4w-0805-surface-mount-chip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; Price (none) -> 0.54
- R8: renamed from R3; footprint Resistor_SMD:R_0805_2012Metric_Pad1.20x1.40mm_HandSolder -> Resistor_SMD:R_1206_3216Metric_Pad1.30x1.75mm_HandSolder; Link (none) -> https://robu.in/product/rl1206fr-070r068l-yageo-250mw-thick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; Price (none) -> 2.08
- R9: renamed from R4; Link (none) -> https://robu.in/product/rc0805fr-07100rl-yageo-res-thick-fi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; Price (none) -> 0.35
- SW1: renamed from SW3; Link (none) -> https://robu.in/product/ss-12f21g5-slide-1p2t-angled-switch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; Price (none) -> 2.50
- U1: renamed from U6; Link (none) -> https://ifuturetech.org/product/mp2307-3a-23v-340khz-synchr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; Price None -> 40
- U2: Link (none) -> http://robu.in/product/tp5100-toppower-5v12v-lithium-ion-po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; Price (none) -> 67
- U3: renamed from U1; Link (none) -> https://robu.in/product/ld1117s50tr-stmicroelectronics-volt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; Price (none) -> 17
- U4: Link (none) -> https://robu.in/product/ld1117s50tr-stmicroelectronics-volt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; Price (none) -> 17
- U5: renamed from U3; Link (none) -> https://robu.in/product/hy2120-cb-hycon-tech-1-5v10v-lithiu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; Price (none) -> 21
- renumbered C1 to C10, C3 to C11, C2 to C12, C4 to C13, C7 to C14, C8 to C15, C10 to C9, D1 to D4, R5 to R10, R6 to R11
Connections:
- net +3V8: now also C22.1
- net GND: now also C22.2
- net at D4.1 (K), U2.2 (LX), U2.3 (LX): now also U10.1
- net at C10.1, C12.1, R8.1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: now also U10.2
