File: kicad/untitled.kicad_sch (KiCad schematic)
At the start: 30 parts, among them J3 Conn_Coaxial, J4 Conn_Coaxial, J5 SIM_Card, J6 Conn_02x20_Odd_Even, J7 Screw_Terminal_01x04, J8 Micro_SD_Card, Q3 NPN, SW1 SW_Push, SW2 SW_Push, U10 MAX3485, U5 ESP32-S3-WROOM-1, U7 SIM7080G, U8 TXS0102DCT

Commit message: update
Parts:
- removed C16: 100nF, Capacitor_SMD:C_0805_2012Metric_Pad1.18x1.45mm_HandSolder, symbol Device:C
- removed J5: SIM_Card, Connector_Card:nanoSIM_GCT_SIM8060-6-0-14-00, symbol Connector:SIM_Card
- removed J8: Micro_SD_Card, Connector_Card:microSD_HC_Wuerth_693072010801, symbol Connector:Micro_SD_Card
- added C18: 100nF, Capacitor_SMD:C_0805_2012Metric_Pad1.18x1.45mm_HandSolder, symbol Device:C
- added Card1: SMN-305, easyeda2kicad:SIM-SMD_SMN-305, symbol easyeda2kicad:SMN-305
- added Card2: THD2528-11SD-GF, easyeda2kicad:TF-SMD_THD2528-11SD-GF, symbol easyeda2kicad:THD2528-11SD-GF
- C19: renamed from C13; Link (none) -> https://robu.in/product/1uf-1000nf-50v-capacitor-0805-smd-p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; Price (none) -> 2.09
- C20: renamed from C14; Link (none) -> https://evelta.com/100uf-6-3v-10-case-b-tantalum-capacitor-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; Price (none) -> 39
- D5: value LED -> R
- D6: value LED -> G
- J4: renamed from J7; Link (none) -> https://robu.in/product/4-pin-5-08mm-pitch-pluggable-screw-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; Price (none) -> 19
- J5: renamed from J6; Link (none) -> https://robu.in/product/2-54mm-pitch-40-pin-male-double-row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; Price (none) -> 12
- J8: renamed from J4; Link (none) -> https://robu.in/product/sma-female-straight-edge-pcb-mount-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; Price (none) -> 65
- Q3: Link (none) -> https://robu.in/product/mmbt2222-npn-transistor-pack-of-15/; Price (none) -> 2.10
- R16: renamed from R11; Link (none) -> https://robu.in/product/crcw080510r0fkeahp-vishay-smd-chip-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; Price (none) -> 3.87
- R19: renamed from R15; Link (none) -> https://robu.in/product/rc0805fr-07330rl-yageo-res-thick-fi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; Price (none) -> 0.80
- SW2: renamed from SW1; footprint Button_Switch_SMD:SW_Push_1P1T_NO_CK_KSC6xxG -> Button_Switch_SMD:SW_Tactile_SPST_NO_Straight_CK_PTS636Sx25SMTRLFS; Link (none) -> https://robu.in/product/362-5mm-tactile-push-button-switch-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; Price (none) -> 3.81
- SW3: renamed from SW2; footprint Button_Switch_SMD:SW_Push_1P1T_NO_CK_KSC6xxG -> Button_Switch_SMD:SW_Tactile_SPST_NO_Straight_CK_PTS636Sx25SMTRLFS; Link (none) -> https://robu.in/product/362-5mm-tactile-push-button-switch-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; Price (none) -> 3.81
- U6: renamed from U5; value ESP32-S3-WROOM-1 -> ESP32-S3-WROOM-1U; Link (none) -> https://evelta.com/esp32-s3-wroom-1u-n16r8-wi-fi-ble-module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; Price (none) -> 325
- U7: renamed from U8; Link (none) -> https://robu.in/product/txs0102dctt-texas-instruments-2-3v5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; Price (none) -> 52
- U8: renamed from U10; Link (none) -> https://robu.in/product/max3485esat-analog-devices-inc-maxi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; Price (none) -> 218
- U9: renamed from U7; Availability In Stock -> (none); Check_prices https://www.snapeda.com/parts/SIM7080G/SIMCom/view-part/?re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 -> (none); Description_1 Cellular, Navigation Galileo, GLONASS, GPS, GNSS, LTE Trans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 -> (none); Link (none) -> https://www.digikey.in/en/products/detail/simcom-wireless-s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; MANUFACTURER SIMCOM -> (none); MAXIMUM_PACKAGE_HEIGHT 2.6 mm -> (none); MF SIMCom -> (none); MP SIM7080G -> (none); PARTREV 1.04 -> (none); Package Package -> (none); Price None -> 2225; STANDARD Manufacturer Recommendation -> (none); SnapEDA_Link https://www.snapeda.com/parts/SIM7080G/SIMCom/view-part/?re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 -> (none)
- renumbered C11 to C16, C12 to C17, C15 to C21, J3 to J6, R8 to R13, R13 to R14, R14 to R15, R9 to R17, R10 to R18, R16 to R20
Connections:
- net +3V3: now also C18.1, Card2.4 (VDD)
- net GND: now also C18.2, Card1.1 (EP), Card1.2 (EP), Card1.3 (EP), Card1.4 (EP), Card1.C5 (GND), Card2.10 (SHELL), Card2.11 (SHELL), Card2.12 (SHELL), Card2.13 (SHELL), Card2.6 (VSS)
- net IO41: now also Card2.2 (CD/DAT3)
- net IO42: now also Card2.3 (CMD)
- net IO47: now also Card2.7 (DAT0)
- net IO48: now also Card2.5 (CLX)
- net SIM_CLK: now also Card1.C3 (CLK)
- net SIM_DATA: now also Card1.C7 (I/O)
- net SIM_RST: now also Card1.C2 (RST)
- net SIM_VDD: now also Card1.C1 (VCC)
- no-connect marks 48 -> 49
