File: kicad/kicad.kicad_pcb (KiCad board)
At the start: 4 copper layers, 88.3 x 112.3 mm, 77 parts, among them J1 USB_C_Receptacle_USB2.0_16P, J2 Barrel_Jack_MountingPin, J3 Conn_Coaxial, J4 Conn_Coaxial, J5 SIM_Card, J6 Conn_02x20_Odd_Even, J7 Screw_Terminal_01x04, J8 Micro_SD_Card, Q1 NMOS, Q2 NMOS, Q3 NPN, SW1 SW_Push, SW2 SW_Push, SW3 SW_SPST, U1 LD1117S50TR_SOT223, U10 MAX3485, U2 TP5100, U3 HY2120, U4 LD1117S33TR_SOT223, U5 ESP32-S3-WROOM-1, U6 MP2307, U7 SIM7080G, U8 TXS0102DCT

Commit message: update
Parts:
- removed ? (x3): , 
- removed the C16 at (192.0, 69.2)
- removed C25: 12uF, Capacitor_SMD:C_0805_2012Metric_Pad1.18x1.45mm_HandSolder
- removed the J5 at (202.8, 104.4)
- removed the J8 at (201.9, 56.8)
- removed the L1 at (161.8, 127.7)
- added C18: 100nF, Capacitor_SMD:C_0805_2012Metric_Pad1.18x1.45mm_HandSolder, F.Cu at (191.3, 53.9)
- added C22: 22 uF, Capacitor_SMD:CP_Elec_5x5.3, F.Cu at (128.4, 105.8)
- added Card1: SMN-305, easyeda2kicad:SIM-SMD_SMN-305, F.Cu at (202.4, 104.6)
- added Card2: THD2528-11SD-GF, easyeda2kicad:TF-SMD_THD2528-11SD-GF, F.Cu at (202.2, 55.6)
- added U10: CDRH104R-220NC, easyeda2kicad:IND-SMD_L10.2-W10.0_SRR1050HA, F.Cu at (161.3, 127.8)
- C2: renamed from C24; value 0.1uF -> 100nF
- D5: value LED -> R
- D6: value LED -> G
- L1: renamed from L3; footprint Inductor_SMD:L_10.4x10.4_H4.8 -> easyeda2kicad:IND-SMD_L10.2-W10.0_SRR1050HA
- R8: renamed from R3; footprint Resistor_SMD:R_0805_2012Metric_Pad1.20x1.40mm_HandSolder -> Resistor_SMD:R_1206_3216Metric_Pad1.30x1.75mm_HandSolder
- SW2: renamed from SW1; footprint Button_Switch_SMD:SW_Push_1P1T_NO_CK_KSC6xxG -> Button_Switch_SMD:SW_Tactile_SPST_NO_Straight_CK_PTS636Sx25SMTRLFS
- SW3: renamed from SW2; footprint Button_Switch_SMD:SW_Push_1P1T_NO_CK_KSC6xxG -> Button_Switch_SMD:SW_Tactile_SPST_NO_Straight_CK_PTS636Sx25SMTRLFS
- U6: renamed from U5; value ESP32-S3-WROOM-1 -> ESP32-S3-WROOM-1U
- renumbered BT2 to BT1, BT1 to BT2, C23 to C1, C1 to C10, C3 to C11, C2 to C12, C4 to C13, C7 to C14, C8 to C15, C11 to C16, C12 to C17, C13 to C19, C14 to C20, C15 to C21, C26 to C3, C19 to C4, C5 to C6, C6 to C7, C9 to C8, C10 to C9, D4 to D1, D1 to D4, J7 to J4, J6 to J5, J3 to J6, J4 to J8, R23 to R1, R5 to R10, R6 to R11, R8 to R13, R13 to R14, R14 to R15, R11 to R16, R9 to R17, R10 to R18, R15 to R19, R1 to R2, R16 to R20, R2 to R3, R28 to R4, R26 to R5, R24 to R6, R4 to R9, SW3 to SW1, U6 to U1, U1 to U3, U3 to U5, U8 to U7, U10 to U8, U7 to U9
Routing:
- net /MCU/IO47: track 81.7 -> 60.3 mm, vias 2 -> 4
- net +3V3: track 260.5 -> 280.1 mm, vias 6 -> 7
- net /MCU/IO42: track 72.0 -> 63.2 mm
- net /MCU/IO41: track 43.3 -> 50.9 mm
- net /MCU/EN: track 49.0 -> 41.6 mm
- net /MCU/IO0: track 58.2 -> 51.5 mm
- net +3V8: track 131.2 -> 129.5 mm
- net VCC: track 112.5 -> 112.0 mm
- net /MCU/IO48: track 56.8 -> 56.7 mm, vias 3 -> 5
- net GND: vias 89 -> 92
Other:
- board text added: "SOILMETRICS v2"
- board text removed: "SOILMETRICS v3"
